File: assets/KiCad/led dot matrix display.sch (KiCad schematic (older format))
At the start: 1 part

Commit message: update some schematics
Parts:
- added Q? (x16): PN2222A, Package_TO_SOT_THT:TO-92_Inline, symbol Transistor_BJT:PN2222A
- added R? (x16): 330, symbol Device:R
Connections:
- net labels added: GND, S0, S1, S10, S11, S12, S13, S14, S15, S2, S3, S4, S5, S6, S7, S8, S9, VCC
- wire segments 0 -> 98
Other:
- moved on the sheet: U?
