File: assets/KiCad/controller.sch (KiCad schematic (older format))
At the start: 0 parts

Commit message: update schematic
Parts:
- added U?: AT128A-70B, symbol MyICs:AT128A-70B
Connections:
- new net C0: U?.30 (PC0)
- new net C1: U?.31 (PC1)
- new net C10: U?.24 (PD2)
- new net C11: U?.25 (PD3)
- new net C12: U?.26 (PD4)
- new net C13: U?.27 (PD5)
- new net C14: U?.28 (PD6)
- new net C15: U?.29 (PD7)
- new net C2: U?.32 (PC2)
- new net C3: U?.33 (PC3)
- new net C4: U?.34 (PC4)
- new net C5: U?.35 (PC5)
- new net C6: U?.36 (PC6)
- new net C7: U?.37 (PC7)
- new net C8: U?.22 (PD0)
- new net C9: U?.23 (PD1)
- new net DA1: U?.11 (PB0)
- new net DA2: U?.12 (PB1)
- new net DA3: U?.13 (PB2)
- new net DA4: U?.14 (PB3)
- new net DB1: U?.15 (PB4)
- new net DB2: U?.16 (PB5)
- new net DB3: U?.17 (PB6)
- new net DB4: U?.18 (PB7)
Changed lines of the file:
@@
 $Descr A4 11693 8268
 encoding utf-8
-Sheet 1 8
+Sheet 5 8
 Title ""
 Date ""
@@
 Comment4 ""
 $EndDescr
+$Comp
+L MyICs:AT128A-70B U?
+U 1 1 5F5DCF09
+P 6000 3900
+F 0 "U?" H 5975 5475 50  0000 C CNN
+F 1 "AT128A-70B" H 5975 5384 50  0000 C CNN
+F 2 "" H 5950 5050 50  0001 C CNN
+F 3 "" H 5950 5050 50  0001 C CNN
+	1    6000 3900
+	1    0    0    -1
+$EndComp
+Wire Wire Line
+	5400 3550 5000 3550
+Wire Wire Line
+	5000 3650 5400 3650
+Wire Wire Line
+	5000 3750 5400 3750
+Wire Wire Line
+	5000 3850 5400 3850
+Wire Wire Line
+	5000 3950 5400 3950
+Wire Wire Line
+	5000 4050 5400 4050
+Wire Wire Line
+	5000 4150 5400 4150
+Wire Wire Line
+	5000 4250 5400 4250
+Wire Wire Line
+	6600 5350 7000 5350
+Wire Wire Line
+	7000 5250 6600 5250
+Wire Wire Line
+	7000 5150 6600 5150
+Wire Wire Line
+	7000 5050 6600 5050
+Wire Wire Line
+	7000 4950 6600 4950
+Wire Wire Line
+	7000 4850 6600 4850
+Wire Wire Line
+	7000 4750 6600 4750
+Wire Wire Line
+	7000 4650 6600 4650
+Wire Wire Line
+	5000 4750 5400 4750
+Wire Wire Line
+	5000 4650 5400 4650
+Wire Wire Line
+	5000 4850 5400 4850
+Wire Wire Line
+	5000 4950 5400 4950
+Wire Wire Line
+	5000 5050 5400 5050
+Wire Wire Line
+	5000 5150 5400 5150
+Wire Wire Line
+	5000 5250 5400 5250
+Wire Wire Line
+	5000 5350 5400 5350
+Text HLabel 5000 3550 0    50   Output ~ 0
+DA1
+Text HLabel 5000 3650 0    50   Output ~ 0
+DA2
+Text HLabel 5000 3750 0    50   Output ~ 0
+DA3
+Text HLabel 5000 3850 0    50   Output ~ 0
+DA4
+Text HLabel 5000 3950 0    50   Output ~ 0
+DB1
+Text HLabel 5000 4050 0    50   Output ~ 0
+DB2
+Text HLabel 5000 4150 0    50   Output ~ 0
+DB3
+Text HLabel 5000 4250 0    50   Output ~ 0
+DB4
+Text HLabel 7000 5350 2    50   Input ~ 0
+C0
+Text HLabel 7000 5250 2    50   Input ~ 0
+C1
+Text HLabel 7000 5150 2    50   Input ~ 0
+C2
+Text HLabel 7000 5050 2    50   Input ~ 0
+C3
+Text HLabel 7000 4950 2    50   Input ~ 0
+C4
+Text HLabel 7000 4850 2    50   Input ~ 0
+C5
+Text HLabel 7000 4750 2    50   Input ~ 0
+C6
+Text HLabel 7000 4650 2    50   Input ~ 0
+C7
+Text HLabel 5000 4650 0    50   Input ~ 0
+C8
+Text HLabel 5000 4750 0    50   Input ~ 0
+C9
+Text HLabel 5000 4850 0    50   Input ~ 0
+C10
+Text HLabel 5000 4950 0    50   Input ~ 0
+C11
+Text HLabel 5000 5050 0    50   Input ~ 0
+C12
+Text HLabel 5000 5150 0    50   Input ~ 0
+C13
+Text HLabel 5000 5250 0    50   Input ~ 0
+C14
+Text HLabel 5000 5350 0    50   Input ~ 0
+C15
 $EndSCHEMATC
