File: assets/KiCad/driver-a.sch (KiCad schematic (older format))
At the start: 33 parts

Commit message: Schematic final
Changed lines of the file:
@@
 Text HLabel 10300 4700 2    50   Output ~ 0
 L15
+Wire Wire Line
+	1550 4750 1450 4750
+Wire Wire Line
+	1450 4750 1450 4850
 Wire Bus Line
 	10000 4100 10000 6200
@@
 Wire Bus Line
 	10000 900  10000 3000
+Connection ~ 1450 4850
 $EndSCHEMATC

Commit message: schematic update
Connections:
- net INH: now reaches U?.23 (INH)
Changed lines of the file:
@@
 L15
 Wire Wire Line
-	1550 4750 1450 4750
-Wire Wire Line
-	1450 4750 1450 4850
+	1200 3700 1550 3700
 Wire Bus Line
 	10000 4100 10000 6200
@@
 Wire Bus Line
 	10000 900  10000 3000
-Connection ~ 1450 4850
+Text HLabel 1200 3700 0    50   Input ~ 0
+INH
 $EndSCHEMATC

Commit message: update schematics
Parts:
- gave numbers to parts that had none: 33
