File: assets/KiCad/driver-b.sch (KiCad schematic (older format))
At the start: 33 parts

Commit message: Schematic final
Changed lines of the file:
@@
 $Descr A4 11693 8268
 encoding utf-8
-Sheet 4 8
+Sheet 8 8
 Title ""
 Date ""
@@
 Text HLabel 10300 4650 2    50   Output ~ 0
 L15
+Wire Wire Line
+	1550 4700 1450 4700
+Wire Wire Line
+	1450 4700 1450 4800
 Wire Bus Line
 	10000 4050 10000 6150
@@
 Wire Bus Line
 	10000 850  10000 2950
+Connection ~ 1450 4800
 $EndSCHEMATC

Commit message: schematic update
Connections:
- net INH: now reaches U?.23 (INH)
Changed lines of the file:
@@
 Text HLabel 10300 4650 2    50   Output ~ 0
 L15
+Text HLabel 1200 3650 0    50   Input ~ 0
+INH
 Wire Wire Line
-	1550 4700 1450 4700
-Wire Wire Line
-	1450 4700 1450 4800
+	1200 3650 1550 3650
 Wire Bus Line
 	10000 4050 10000 6150
@@
 Wire Bus Line
 	10000 850  10000 2950
-Connection ~ 1450 4800
 $EndSCHEMATC

Commit message: update schematics
Parts:
- gave numbers to parts that had none: 33
Other:
- moved on the sheet: Q17, Q18, Q19, Q20, Q21, Q22, Q23, Q24, Q25, Q26, Q27, Q28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
