File: assets/KiCad/led matrix.sch (KiCad schematic (older format))
At the start: 3 parts

Commit message: minor update
Parts:
- removed J? (x3): Conn_01x16, symbol Connector_Generic:Conn_01x16
Connections:
- net labels added: C0, C1, C10, C11, C12, C13, C14, C15, C2, C3, C4, C5, C6, C7, C8, C9, DA0, DA1, DA10, DA11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
- wire segments 0 -> 96
