File: assets/KiCad/led-b.sch (KiCad schematic (older format))
At the start: 256 parts

Commit message: update schematics
Parts:
- gave numbers to parts that had none: 256
Other:
- moved on the sheet: D257, D258, D259, D260, D261, D262, D263, D264, D265, D266, D267, D268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
